File: circuit/main/main.kicad_sch (KiCad schematic)
At the start: 1 part, among them U1 STM32F405RGTx

Commit message: 回路すすめた
Parts:
- added C1, C2: 2.2u, symbol Device:C_Small
- added C10, C3, C4, C5, C6, C7, C8, C9: 0.1u, symbol Device:C_Small
- added FB1: FerriteBead_Small, symbol Device:FerriteBead_Small
- added J1: Conn_01x06, symbol Connector_Generic:Conn_01x06
- added J2, J3: Conn_02x05_Odd_Even, symbol Connector_Generic:Conn_02x05_Odd_Even
- added R1: R, symbol Device:R
- added SW1: SW_Push, symbol Switch:SW_Push
- added U2: ~, symbol mylib:OSC
Connections:
- net +3.3V: now reaches U1.1 (VBAT)
- net +3.3V: now also U1.19 (VDD), U1.32 (VDD), U1.48 (VDD), U1.64 (VDD), C4.1, C5.1, C6.1, C7.1, C8.1, C9.1, FB1.1, J1.1 (Pin_1), U2.8 (VDD)
- net GNDA: now reaches U1.12 (VSSA)
- net GNDA: now also C10.2
- net VDDA: now reaches U1.13 (VDDA)
- net VDDA: now also C10.1, FB1.2
- net GND: now reaches U1.18 (VSS), U1.63 (VSS)
- net GND: now also C1.2, C2.2, C3.2, C4.2, C5.2, C6.2, C7.2, C8.2, C9.2, J1.3 (Pin_3), J2.3 (Pin_3), J3.3 (Pin_3), R1.2, SW1.1, U2.4 (GND)
- net at U1.31 (VCAP_1): now also C2.1
- net at U1.47 (VCAP_2): now also C1.1
- net at U1.5 (PH0): now also U2.5 (Output)
- net at U1.60 (BOOT0): now also R1.1
- net at U1.7 (NRST): now also C3.1, J1.5 (Pin_5), SW1.2
- new net +5V: J2.2 (Pin_2), J3.2 (Pin_2)
- new net ENC1_A: J2.6 (Pin_6)
- new net ENC1_B: J2.8 (Pin_8)
- new net ENC2_A: J3.6 (Pin_6)
- new net ENC2_B: J3.8 (Pin_8)
- new net SWCLC: J1.2 (Pin_2)
- new net SWDIO: J1.4 (Pin_4)
- new net SWO: J1.6 (Pin_6)
- no-connect marks 0 -> 14
