File: 2024_robotracer_circuit/following_sensor/following_sensor.kicad_pcb (KiCad board)
At the start: 2 copper layers, 88 x 14 mm, 14 parts, among them J1 PH_8p, U1 LBR-127HLD, U2 LBR-127HLD, U3 LBR-127HLD, U4 LBR-127HLD

Commit message: サイドセンサ
Parts:
- added G***: LOGO, mylib:SH_5mm, B.Cu at (159.5, 92.0)
