File: 2024_robotracer_circuit/following_sensor/following_sensor.kicad_sch (KiCad schematic)
At the start: 15 parts, among them J1 PH_8p, U1 LBR-127HLD, U2 LBR-127HLD, U3 LBR-127HLD, U4 LBR-127HLD

Commit message: センサー
Parts:
- removed C1: 0.1u, Capacitor_SMD:C_0603_1608Metric_Pad1.08x0.95mm_HandSolder, symbol Device:C_Small
Changed lines of the file:
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@@
-	)
-	(junction
-		(at 83.82 86.36)
-		(diameter 0)
-		(color 0 0 0 0)
 	)
 	(junction
@@
 	)
 	(junction
-		(at 71.12 55.88)
-		(diameter 0)
-		(color 0 0 0 0)
-	)
-	(junction
 		(at 62.23 86.36)
 		(diameter 0)
@@
 	(wire
 		(pts
-			(xy 83.82 55.88) (xy 71.12 55.88)
-		)
-		(stroke
-			(width 0)
-			(type default)
-		)
-	)
-	(wire
-		(pts
 			(xy 218.44 118.11) (xy 218.44 120.65)
 		)
@@
 	(wire
 		(pts
-			(xy 92.71 86.36) (xy 83.82 86.36)
-		)
-		(stroke
-			(width 0)
-			(type default)
-		)
-	)
-	(wire
-		(pts
-			(xy 83.82 78.74) (xy 83.82 55.88)
+			(xy 62.23 86.36) (xy 92.71 86.36)
 		)
 		(stroke
@@
 	(wire
 		(pts
-			(xy 83.82 83.82) (xy 83.82 86.36)
-		)
-		(stroke
-			(width 0)
-			(type default)
-		)
-	)
-	(wire
-		(pts
 			(xy 190.5 110.49) (xy 198.12 110.49)
-		)
-		(stroke
-			(width 0)
-			(type default)
-		)
-	)
-	(wire
-		(pts
-			(xy 83.82 86.36) (xy 62.23 86.36)
 		)
 		(stroke
@@
 					(unit 1)
 				)
-			)
-		)
-	)
-	(symbol
-		(lib_id "Device:C_Small")
-		(at 83.82 81.28 0)
-		(mirror y)
-		(unit 1)
-		(exclude_from_sim no)
-		(in_bom yes)
-		(on_board yes)
-		(dnp no)
-		(fields_autoplaced yes)
-		(property "Reference" "C1"
-			(at 81.28 80.0162 0)
-			(effects
-				(font
-					(size 1.27 1.27)
-				)
-				(justify left)
-			)
-		)
-		(property "Value" "0.1u"
-			(at 81.28 82.5562 0)
-			(effects
-				(font
-					(size 1.27 1.27)
-				)
-				(justify left)
-			)
-		)
-		(property "Footprint" "Capacitor_SMD:C_0603_1608Metric_Pad1.08x0.95mm_HandSolder"
-			(at 83.82 81.28 0)
-			(effects
-				(font
-					(size 1.27 1.27)
-				)
-				(hide yes)
-			)
-		)
-		(property "Datasheet" "~"
-			(at 83.82 81.28 0)
-			(effects
-				(font
-					(size 1.27 1.27)
-				)
-				(hide yes)
-			)
-		)
-		(property "Description" "Unpolarized capacitor, small symbol"
-			(at 83.82 81.28 0)
-			(effects
-				(font
-					(size 1.27 1.27)
-				)
-				(hide yes)
-			)
-		)
-		(pin "2"
-		)
-		(pin "1"
-		)
-		(instances
-			(project "following_sensor"
-				(path "/542d1ff3-a6c0-4d9d-8de4-1794f2b50dfd"
-					(reference "C1")
-					(unit 1)
-				)

Commit message: hoge
Parts:
- R1, R2, R3, R4: value 4.7 -> 5.1
Changed lines of the file:
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@@
 			)
 		)
-		(property "Value" "4.7"
+		(property "Value" "5.1"
 			(at 220.98 124.4599 0)
 			(effects
@@
 			)
 		)
-		(property "Value" "4.7"
+		(property "Value" "5.1"
 			(at 177.8 124.4599 0)
 			(effects
@@
 			)
 		)
-		(property "Value" "4.7"
+		(property "Value" "5.1"
 			(at 132.08 124.4599 0)
 			(effects
@@
 			)
 		)
-		(property "Value" "4.7"
+		(property "Value" "5.1"
 			(at 85.09 124.4599 0)
 			(effects

Commit message: デバッグ用無限ループ削除
Parts:
- R5: value R_Small -> 1.8k
- R6: value R_Small -> 3k
Changed lines of the file:
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@@
 			)
 		)
-		(property "Value" "R_Small"
+		(property "Value" "1.8k"
 			(at 154.94 68.5799 0)
 			(effects
@@
 			)
 		)
-		(property "Value" "R_Small"
+		(property "Value" "3k"
 			(at 177.8 68.5799 0)
 			(effects
