File: 2024_robotracer_circuit/main/main.kicad_pcb (KiCad board)
At the start: 2 copper layers, 60 x 60 mm, 70 parts, among them J1 PH_6p, J10 PH_5p, J11 PH_6p, J13 PH_8p, J2 Conn_02x05_Odd_Even, J3 Conn_02x05_Odd_Even, J4 PA_2p, J5 PA_2p, J6 XT_2p, J7 HX_12p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

Commit message: 修正
Parts:
- moved J10 3.00 mm to (119.0, 81.5)
- moved R5 2.88 mm to (121.6, 78.3)
Routing:
- net GND: track 523.2 -> 530.4 mm, vias 115 -> 118
- net Net-(J10-Pin_4): track 62.8 -> 60.5 mm
- net /SENSOR_L_ADC: track 17.6 -> 18.5 mm
- net +BATT: track 140.6 -> 139.7 mm
- net +3.3V: track 371.8 -> 372.3 mm

Commit message: 製造ファイル生成
Parts:
- added REF**: MountingHole_2.2mm_M2, MountingHole:MountingHole_2.2mm_M2, F.Cu at (156.0, 96.0)
- added REF**: MountingHole_2.2mm_M2, MountingHole:MountingHole_2.2mm_M2, F.Cu at (100.0, 40.0)
- added REF**: MountingHole_2.2mm_M2, MountingHole:MountingHole_2.2mm_M2, F.Cu at (100.0, 96.0)
- added REF**: MountingHole_2.2mm_M2, MountingHole:MountingHole_2.2mm_M2, F.Cu at (156.0, 40.0)
