File: 2024_robotracer_circuit/sd_card/sd_card.kicad_sch (KiCad schematic)
At the start: 11 parts, among them J1 Micro_SD_Card_Det1, J2 PH_6p

Commit message: sdカード
Parts:
- removed C1: 100u, Capacitor_SMD:CP_Elec_6.3x5.4, symbol Device:C_Polarized_Small
- added C1: 0.1u, Capacitor_SMD:C_0603_1608Metric_Pad1.08x0.95mm_HandSolder, symbol Device:C_Small
Connections:
- net +3.3V: now also C1.1
- net GND: now also C1.2
- net SDIO_CK: now also J2.4 (Pin_4); no longer J2.3 (Pin_3)
- net SDIO_CMD: now also J2.5 (Pin_5); no longer J2.2 (Pin_2)
- net SDIO_D0: now also J2.2 (Pin_2); no longer J2.4 (Pin_4)
- net SDIO_SW: now also J2.3 (Pin_3); no longer J2.5 (Pin_5)
Changed lines of the file:
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@@
 	)
 	(label "SDIO_CMD"
-		(at 74.93 45.72 0)
+		(at 74.93 53.34 0)
 		(fields_autoplaced yes)
 		(effects
@@
 	)
 	(label "SDIO_SW"
-		(at 74.93 53.34 0)
+		(at 74.93 48.26 0)
 		(fields_autoplaced yes)
 		(effects
@@
 	)
 	(label "SDIO_CK"
-		(at 74.93 48.26 0)
+		(at 74.93 50.8 0)
 		(fields_autoplaced yes)
 		(effects
@@
 	)
 	(label "SDIO_D0"
-		(at 74.93 50.8 0)
+		(at 74.93 45.72 0)
 		(fields_autoplaced yes)
 		(effects
@@
 	)
 	(symbol
-		(lib_id "Device:C_Polarized_Small")
-		(at 107.95 110.49 0)
-		(mirror y)
-		(unit 1)
-		(exclude_from_sim no)
-		(in_bom yes)
-		(on_board yes)
-		(dnp no)
-		(fields_autoplaced yes)
-		(property "Reference" "C1"
-			(at 110.49 108.6738 0)
-			(effects
-				(font
-					(size 1.27 1.27)
-				)
-				(justify right)
-			)
-		)
-		(property "Value" "100u"
-			(at 110.49 111.2138 0)
-			(effects
-				(font
-					(size 1.27 1.27)
-				)
-				(justify right)
-			)
-		)
-		(property "Footprint" "Capacitor_SMD:CP_Elec_6.3x5.4"
-			(at 107.95 110.49 0)
-			(effects
-				(font
-					(size 1.27 1.27)
-				)
-				(hide yes)
-			)
-		)
-		(property "Datasheet" "~"
-			(at 107.95 110.49 0)
-			(effects
-				(font
-					(size 1.27 1.27)
-				)
-				(hide yes)
-			)
-		)
-		(property "Description" "Polarized capacitor, small symbol"
-			(at 107.95 110.49 0)
-			(effects
-				(font
-					(size 1.27 1.27)
-				)
-				(hide yes)
-			)
-		)
-		(pin "1"
-		)
-		(pin "2"
-		)
-		(instances
-			(project "sd_card"
-				(path "/5c8bc54e-35dd-4c32-851e-a2e69654c7d1"
-					(reference "C1")
-					(unit 1)
-				)
-			)
-		)
-	)
-	(symbol
 		(lib_id "power:PWR_FLAG")
 		(at 83.82 55.88 0)
@@
 					(unit 1)
 				)
+			)
+		)
+	)
+	(symbol
+		(lib_id "Device:C_Small")
+		(at 107.95 110.49 0)
+		(mirror y)
+		(unit 1)
+		(exclude_from_sim no)
+		(in_bom yes)
+		(on_board yes)
+		(dnp no)
+		(fields_autoplaced yes)
+		(property "Reference" "C1"
+			(at 110.49 109.2262 0)
+			(effects
+				(font
+					(size 1.27 1.27)
+				)
+				(justify right)
+			)
+		)
+		(property "Value" "0.1u"
+			(at 110.49 111.7662 0)
+			(effects
+				(font
+					(size 1.27 1.27)
+				)
+				(justify right)
+			)
+		)
+		(property "Footprint" "Capacitor_SMD:C_0603_1608Metric_Pad1.08x0.95mm_HandSolder"
+			(at 107.95 110.49 0)
+			(effects
+				(font
+					(size 1.27 1.27)
+				)
+				(hide yes)
+			)
+		)
+		(property "Datasheet" "~"
+			(at 107.95 110.49 0)
+			(effects
+				(font
+					(size 1.27 1.27)
+				)
+				(hide yes)
+			)
+		)
+		(property "Description" "Unpolarized capacitor, small symbol"
+			(at 107.95 110.49 0)
+			(effects
+				(font
+					(size 1.27 1.27)
+				)
+				(hide yes)
+			)
+		)
+		(pin "1"
+		)
+		(pin "2"
+		)
+		(instances
+			(project "sd_card"
+				(path "/5c8bc54e-35dd-4c32-851e-a2e69654c7d1"
+					(reference "C1")
+					(unit 1)
+				)
