File: 2024_robotracer_circuit/side_sensor/side_sensor.kicad_sch (KiCad schematic)
At the start: 9 parts, among them J2 PH_5p, U1 LBR-127HLD

Commit message: サイドセンサ
Parts:
- removed C1: 0.1u, Capacitor_SMD:C_0603_1608Metric_Pad1.08x0.95mm_HandSolder, symbol Device:C_Small
Connections:
- net SENSOR0_ADC is gone; now on net SENSOR_SIDE_ADC: U1.4 (C)
Changed lines of the file:
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@@
 	(paper "A4")
-	(junction
-		(at 92.71 82.55)
-		(diameter 0)
-		(color 0 0 0 0)
-	)
 	(junction
 		(at 71.12 82.55)
@@
 		(color 0 0 0 0)
 	)
-	(junction
-		(at 80.01 59.69)
-		(diameter 0)
-		(color 0 0 0 0)
-	)
 	(wire
 		(pts
@@
 	(wire
 		(pts
-			(xy 92.71 80.01) (xy 92.71 82.55)
-		)
-		(stroke
-			(width 0)
-			(type default)
-		)
-	)
-	(wire
-		(pts
 			(xy 73.66 67.31) (xy 73.66 69.85)
 		)
@@
 	(wire
 		(pts
-			(xy 92.71 59.69) (xy 80.01 59.69)
-		)
-		(stroke
-			(width 0)
-			(type default)
-		)
-	)
-	(wire
-		(pts
-			(xy 92.71 82.55) (xy 71.12 82.55)
+			(xy 71.12 82.55) (xy 101.6 82.55)
 		)
 		(stroke
@@
 	(wire
 		(pts
-			(xy 101.6 82.55) (xy 92.71 82.55)
-		)
-		(stroke
-			(width 0)
-			(type default)
-		)
-	)
-	(wire
-		(pts
 			(xy 137.16 115.57) (xy 144.78 115.57)
 		)
@@
 		(pts
 			(xy 184.15 67.31) (xy 184.15 68.58)
-		)
-		(stroke
-			(width 0)
-			(type default)
-		)
-	)
-	(wire
-		(pts
-			(xy 92.71 74.93) (xy 92.71 59.69)
 		)
 		(stroke
@@
 		)
 	)
-	(label "PULSE"
-		(at 66.04 74.93 0)
+	(label "SENSOR_SIDE_ADC"
+		(at 144.78 115.57 0)
 		(fields_autoplaced yes)
 		(effects
@@
 		)
 	)
-	(label "SENSOR0_ADC"
-		(at 144.78 115.57 0)
+	(label "PULSE"
+		(at 66.04 74.93 0)
 		(fields_autoplaced yes)
 		(effects
@@
 					(unit 1)
 				)
-			)
-		)
-	)
-	(symbol
-		(lib_id "Device:C_Small")
-		(at 92.71 77.47 0)
-		(mirror y)
-		(unit 1)
-		(exclude_from_sim no)
-		(in_bom yes)
-		(on_board yes)
-		(dnp no)
-		(fields_autoplaced yes)
-		(property "Reference" "C1"
-			(at 90.17 76.2062 0)
-			(effects
-				(font
-					(size 1.27 1.27)
-				)
-				(justify left)
-			)
-		)
-		(property "Value" "0.1u"
-			(at 90.17 78.7462 0)
-			(effects
-				(font
-					(size 1.27 1.27)
-				)
-				(justify left)
-			)
-		)
-		(property "Footprint" "Capacitor_SMD:C_0603_1608Metric_Pad1.08x0.95mm_HandSolder"
-			(at 92.71 77.47 0)
-			(effects
-				(font
-					(size 1.27 1.27)
-				)
-				(hide yes)
-			)
-		)
-		(property "Datasheet" "~"
-			(at 92.71 77.47 0)
-			(effects
-				(font
-					(size 1.27 1.27)
-				)
-				(hide yes)
-			)
-		)
-		(property "Description" "Unpolarized capacitor, small symbol"
-			(at 92.71 77.47 0)
-			(effects
-				(font
-					(size 1.27 1.27)
-				)
-				(hide yes)
-			)
-		)
-		(pin "2"
-		)
-		(pin "1"
-		)
-		(instances
-			(project "side_sensor"
-				(path "/a42dd4c6-b236-415a-8b71-3f8e0cd98396"
-					(reference "C1")
-					(unit 1)
-				)

Commit message: hoge
Parts:
- R1: value 4.7 -> 5.1
Changed lines of the file:
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@@
 			)
 		)
-		(property "Value" "4.7"
+		(property "Value" "5.1"
 			(at 124.46 129.5399 0)
 			(effects
